Commit message: collision checking and before saving data

File: cpp/RobotModel/valkyrie.urdf (robot description, URDF)
Before this commit: robot valkyrie, 78 links, 77 joints
Links:
- link head: geometry visual mesh filename=meshes/multisense/head.dae
- link hokuyo_link: geometry visual mesh filename=meshes/multisense/head_camera.dae
- link leftAnklePitchLink: geometry visual mesh filename=meshes/legs/lj5.dae
- link leftElbowPitchLink: geometry visual mesh filename=meshes/arms/aj4_left.dae
- link leftHipPitchLink: geometry visual mesh filename=meshes/legs/lj3_left.dae
- link leftHipRollLink: geometry visual mesh filename=meshes/legs/lj2_left.dae
- link leftHipYawLink: geometry visual mesh filename=meshes/legs/lj1_left.dae
- link leftIndexFingerPitch1Link: geometry visual mesh filename=meshes/fingers/indexj1_left.dae
- link leftIndexFingerPitch2Link: geometry visual mesh filename=meshes/fingers/indexj2_left.dae
- link leftIndexFingerPitch3Link: geometry visual mesh filename=meshes/fingers/indexj3_left.dae
- link leftMiddleFingerPitch1Link: geometry visual mesh filename=meshes/fingers/middlej1_left.dae
- link leftMiddleFingerPitch2Link: geometry visual mesh filename=meshes/fingers/middlej2_left.dae
- link leftMiddleFingerPitch3Link: geometry visual mesh filename=meshes/fingers/middlej3_left.dae
- link leftPinkyPitch1Link: geometry visual mesh filename=meshes/fingers/pinkyj1_left.dae
- link leftPinkyPitch2Link: geometry visual mesh filename=meshes/fingers/pinkyj2_left.dae
- link leftPinkyPitch3Link: geometry visual mesh filename=meshes/fingers/pinkyj3_left.dae
- link leftShoulderPitchLink: geometry visual mesh filename=meshes/arms/aj1_left.dae
- link leftShoulderRollLink: geometry visual mesh filename=meshes/arms/aj2_left.dae
- link leftThumbPitch1Link: geometry visual mesh filename=meshes/fingers/thumbj2_left.dae
- link leftThumbPitch2Link: geometry visual mesh filename=meshes/fingers/thumbj3_left.dae
- link leftThumbPitch3Link: geometry visual mesh filename=meshes/fingers/thumbj4_left.dae
- link leftThumbRollLink: geometry visual mesh filename=meshes/fingers/thumbj1_left.dae
- link leftWristRollLink: geometry visual mesh filename=meshes/arms/aj6_left.dae
- link lowerNeckPitchLink: geometry visual mesh filename=meshes/head/neckj1.dae
- link neckYawLink: geometry visual mesh filename=meshes/head/neckj2.dae
- link rightAnklePitchLink: geometry visual mesh filename=meshes/legs/lj5.dae
- link rightElbowPitchLink: geometry visual mesh filename=meshes/arms/aj4_right.dae
- link rightHipPitchLink: geometry visual mesh filename=meshes/legs/lj3_right.dae
- link rightHipRollLink: geometry visual mesh filename=meshes/legs/lj2_right.dae
- link rightHipYawLink: geometry visual mesh filename=meshes/legs/lj1_right.dae
- link rightIndexFingerPitch1Link: geometry visual mesh filename=meshes/fingers/indexj1_right.dae
- link rightIndexFingerPitch2Link: geometry visual mesh filename=meshes/fingers/indexj2_right.dae
- link rightIndexFingerPitch3Link: geometry visual mesh filename=meshes/fingers/indexj3_right.dae
- link rightMiddleFingerPitch1Link: geometry visual mesh filename=meshes/fingers/middlej1_right.dae
- link rightMiddleFingerPitch2Link: geometry visual mesh filename=meshes/fingers/middlej2_right.dae
- link rightMiddleFingerPitch3Link: geometry visual mesh filename=meshes/fingers/middlej3_right.dae
- link rightPinkyPitch1Link: geometry visual mesh filename=meshes/fingers/pinkyj1_right.dae
- link rightPinkyPitch2Link: geometry visual mesh filename=meshes/fingers/pinkyj2_right.dae
- link rightPinkyPitch3Link: geometry visual mesh filename=meshes/fingers/pinkyj3_right.dae
- link rightShoulderPitchLink: geometry visual mesh filename=meshes/arms/aj1_right.dae
- link rightShoulderRollLink: geometry visual mesh filename=meshes/arms/aj2_right.dae
- link rightThumbPitch1Link: geometry visual mesh filename=meshes/fingers/thumbj2_right.dae
- link rightThumbPitch2Link: geometry visual mesh filename=meshes/fingers/thumbj3_right.dae
- link rightThumbPitch3Link: geometry visual mesh filename=meshes/fingers/thumbj4_right.dae
- link rightThumbRollLink: geometry visual mesh filename=meshes/fingers/thumbj1_right.dae
- link rightWristRollLink: geometry visual mesh filename=meshes/arms/aj6_right.dae
- link torsoPitchLink: geometry visual mesh filename=meshes/torso/torsopitch.dae
- link torsoYawLink: geometry visual mesh filename=meshes/torso/torsoyaw.dae
- link upperNeckPitchLink: geometry visual mesh filename=meshes/head/head_multisense_no_visor.dae
